File: RS485_Click/RS485_Click.kicad_sch (KiCad schematic)
At the start: 20 parts, among them J1 RS485, J2 RS485 Click v1.0 by MPro, U2 YD3082EESA

Commit message: project files updated to Kicad version 9.0.1
Parts:
- renumbered D2 to D1, D3 to D2, D4 to D3, D1 to D4, R8 to R1, R9 to R2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
