File: RS485_Click/RS485_Click.kicad_pcb (KiCad board)
At the start: 2 copper layers, 25.4 x 42.9 mm, 23 parts, among them J1 RS485, J2 RS485 Click v1.0 by MPro, U1 YD3082EESA

Commit message: project files updated to Kicad version 9.0.1
Parts:
- J2: value RS485 Click v1.0 by MPro -> RS485 Click v${REVISION} by MPro

Commit message: updated 3D models and project files
Other:
- board text removed: "JLCJLCJLCJLC"
Changed lines of the file:
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@@
 			)
 		)
-		(model "${KIPRJMOD}/shapes3D/Jumper-blue.step"
+		(model "${KIPRJMOD}/shapes3D/Jumper-blue.stpZ"
 			(offset
 				(xyz 0 -3.81 0)
@@
 			)
 		)
-		(model "${KIPRJMOD}/shapes3D/Jumper-red.step"
+		(model "${KIPRJMOD}/shapes3D/Jumper-red.stpZ"
 			(offset
 				(xyz 0 -3.81 0)
@@
 		)
 		(property "Datasheet" ""
-			(at 0 0 270)
+			(at 0 0 90)
 			(layer "F.Fab")
 			(hide yes)
@@
 		)
 		(property "Description" "Jumper, 2-pole, open"
-			(at 0 0 270)
+			(at 0 0 90)
 			(layer "F.Fab")
 			(hide yes)
@@
 			)
 		)
-		(model "${KIPRJMOD}/shapes3D/Jumper-green.step"
+		(model "${KIPRJMOD}/shapes3D/Jumper-green.stpZ"
 			(offset
 				(xyz 0 -1.27 0)
@@
 		)
 		(property "Datasheet" ""
-			(at 0 0 270)
+			(at 0 0 90)
 			(layer "F.Fab")
 			(hide yes)
@@
 		)
 		(property "Description" "Jumper, 2-pole, open"
-			(at 0 0 270)
+			(at 0 0 90)
 			(layer "F.Fab")
 			(hide yes)
@@
 			)
 		)
-		(model "${KIPRJMOD}/shapes3D/Jumper-green.step"
+		(model "${KIPRJMOD}/shapes3D/Jumper-green.stpZ"
 			(offset
 				(xyz 0 -1.27 0)
@@
 		)
 		(property "Datasheet" ""
-			(at 0 0 270)
+			(at 0 0 90)
 			(layer "F.Fab")
 			(hide yes)
@@
 		)
 		(property "Description" "Jumper, 2-pole, open"
-			(at 0 0 270)
+			(at 0 0 90)
 			(layer "F.Fab")
 			(hide yes)
@@
 			)
 		)
-		(model "${KIPRJMOD}/shapes3D/Jumper-yellow.step"
+		(model "${KIPRJMOD}/shapes3D/Jumper-yellow.stpZ"
 			(offset
 				(xyz 0 -1.27 0)
@@
 		)
 	)
-	(gr_text "JLCJLCJLCJLC"
-		(at 94.784786 47.929286 0)
-		(layer "F.SilkS")
-		(effects
-			(font
-				(size 0.81 0.81)
-				(thickness 0.15)
-				(bold yes)
-			)
-			(justify left bottom)
-		)
-	)
 	(gr_text "One pin\nenables"
 		(at 110.913786 55.930286 90)
@@
 			(prefix "")
 			(suffix "")
-			(units 3)
+			(units 2)
 			(units_format 1)
-			(precision 4)
+			(precision 2)
 		)
 		(style
@@
 			(keep_text_aligned yes)
 		)
-		(gr_text "25,4000 mm"
+		(gr_text "25.40 mm"
 			(at 99.102786 37.508286 0)
 			(layer "Dwgs.User")
@@
 			(prefix "")
 			(suffix "")
-			(units 3)
+			(units 2)
 			(units_format 1)
-			(precision 4)
+			(precision 2)
 		)
 		(style
@@
 			(keep_text_aligned yes)
 		)
-		(gr_text "42,9260 mm"
+		(gr_text "42.93 mm"
 			(at 82.712786 62.280286 90)
 			(layer "Dwgs.User")
@@
 			(prefix "")
 			(suffix "")
-			(units 3)
+			(units 2)
 			(units_format 1)
-			(precision 4)
+			(precision 2)
 		)
 		(style
@@
 			(keep_text_aligned yes)
 		)
-		(gr_text "22,8600 mm"
+		(gr_text "22.86 mm"
 			(at 97.832786 85.133286 0)
 			(layer "Dwgs.User")
