File: I2C_EEPROM_Click/I2C_EEPROM_Click.kicad_pcb (KiCad board)
At the start: 2 copper layers, 25.4 x 28.6 mm, 19 parts, among them J1 I^{2}C EEPROM Click v${REVISI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, U1 AT24C256

Commit message: updated 3D models and project files
Other:
- board text removed: "JLCJLCJLCJLC"
Changed lines of the file:
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@@
 		)
 		(embedded_fonts no)
-		(model "${KICAD6_3DMODEL_DIR}/Connector_PinHeader_2.54mm.3dshapes/PinHeader_1x03_P2.54mm_Vertical.wrl"
+		(model "${KIPRJMOD}/shapes3D/PinHeader_1x03_P2.54mm_Vertical.wrl"
 			(offset
 				(xyz 0 0 0)
@@
 			)
 		)
-		(model "${KIPRJMOD}/shapes3D/Jumper-red.step"
+		(model "${KIPRJMOD}/shapes3D/Jumper-red.stpZ"
 			(offset
 				(xyz 0 -3.81 0)
@@
 		)
 		(embedded_fonts no)
-		(model "${KICAD6_3DMODEL_DIR}/Connector_PinHeader_2.54mm.3dshapes/PinHeader_1x03_P2.54mm_Vertical.wrl"
+		(model "${KIPRJMOD}/shapes3D/PinHeader_1x03_P2.54mm_Vertical.wrl"
 			(offset
 				(xyz 0 0 0)
@@
 			)
 		)
-		(model "${KIPRJMOD}/shapes3D/Jumper-blue.step"
+		(model "${KIPRJMOD}/shapes3D/Jumper-blue.stpZ"
 			(offset
 				(xyz 0 -3.81 0)
@@
 		)
 		(embedded_fonts no)
-		(model "${KICAD6_3DMODEL_DIR}/Connector_PinHeader_2.54mm.3dshapes/PinHeader_1x03_P2.54mm_Vertical.wrl"
+		(model "${KIPRJMOD}/shapes3D/PinHeader_1x03_P2.54mm_Vertical.wrl"
 			(offset
 				(xyz 0 0 0)
@@
 			)
 		)
-		(model "${KIPRJMOD}/shapes3D/Jumper-yellow.step"
+		(model "${KIPRJMOD}/shapes3D/Jumper-yellow.stpZ"
 			(offset
 				(xyz 0 -3.81 0)
@@
 		)
 		(embedded_fonts no)
-		(model "${KICAD6_3DMODEL_DIR}/Connector_PinHeader_2.54mm.3dshapes/PinHeader_1x03_P2.54mm_Vertical.wrl"
+		(model "${KIPRJMOD}/shapes3D/PinHeader_1x03_P2.54mm_Vertical.wrl"
 			(offset
 				(xyz 0 0 0)
@@
 			)
 		)
-		(model "${KIPRJMOD}/shapes3D/Jumper-blue.step"
+		(model "${KIPRJMOD}/shapes3D/Jumper-blue.stpZ"
 			(offset
 				(xyz 0 -3.81 0)
@@
 		)
 		(embedded_fonts no)
-		(model "${KICAD6_3DMODEL_DIR}/Connector_PinHeader_2.54mm.3dshapes/PinHeader_1x03_P2.54mm_Vertical.wrl"
+		(model "${KIPRJMOD}/shapes3D/PinHeader_1x03_P2.54mm_Vertical.wrl"
 			(offset
 				(xyz 0 0 0)
@@
 			)
 		)
-		(model "${KIPRJMOD}/shapes3D/Jumper-blue.step"
+		(model "${KIPRJMOD}/shapes3D/Jumper-blue.stpZ"
 			(offset
 				(xyz 0 -3.81 0)
@@
 		(embedded_fonts no)
 	)
-	(gr_text "JLCJLCJLCJLC"
-		(at 107.95 70.485 0)
-		(layer "B.SilkS")
-		(effects
-			(font
-				(size 0.81 0.81)
-				(thickness 0.15)
-				(bold yes)
-			)
-			(justify bottom mirror)
-		)
-	)
 	(dimension
 		(type aligned)
 		(layer "Dwgs.User")
 		(pts
-			(xy 95.0035 78.135) (xy 120.4035 78.135)
+			(xy 95.0035 78.135) (xy 117.8635 78.135)
 		)
-		(height 3.048)
+		(height 2.256)
 		(format
 			(prefix "")
 			(suffix "")
-			(units 3)
+			(units 2)
 			(units_format 1)
-			(precision 4)
+			(precision 2)
 		)
 		(style
@@
 			(keep_text_aligned yes)
 		)
-		(gr_text "25,4000 mm"
-			(at 107.7035 80.033 0)
+		(gr_text "22.86 mm"
+			(at 106.4335 79.241 0)
 			(layer "Dwgs.User")
 			(effects
@@
 			(prefix "")
 			(suffix "")
-			(units 3)
+			(units 2)
 			(units_format 1)
-			(precision 4)
+			(precision 2)
 		)
 		(style
@@
 			(keep_text_aligned yes)
 		)
-		(gr_text "28,5750 mm"
+		(gr_text "28.57 mm"
 			(at 91.56 63.8475 90)
 			(layer "Dwgs.User")
 			(effects
+				(font
+					(size 1 1)
+					(thickness 0.15)
+				)
+			)
+		)
+	)
+	(dimension
+		(type orthogonal)
+		(layer "Dwgs.User")
+		(pts
+			(xy 95.0035 49.56) (xy 120.4035 49.56)
+		)
+		(height -1.935)
+		(orientation 0)
+		(format
+			(prefix "")
+			(suffix "")
+			(units 2)
+			(units_format 1)
+			(precision 2)
+		)
+		(style
+			(thickness 0.15)
+			(arrow_length 1.27)
+			(text_position_mode 0)
+			(arrow_direction outward)
+			(extension_height 0.58642)
+			(extension_offset 0.5)
+			(keep_text_aligned yes)
+		)
+		(gr_text "25.40 mm"
+			(at 107.7035 46.475 0)
+			(layer "Dwgs.User")
+			(effects
