File: Arduino_UNO_click_shield/Arduino_UNO_click_shield.kicad_pcb (KiCad board)
At the start: 2 copper layers, 68.6 x 53.3 mm, 16 parts, among them J1 mikroBUS host connector, J2 mikroBUS host connector, J4 UPDI, U1 ATtiny1616-M

Commit message: project files updated to Kicad version 9.0.1
Connections:
- A1 pad 13: /SDA -> unconnected-(A1-SDA/A4-Pad13)
- A1 pad 14: /SCL -> unconnected-(A1-SCL/A5-Pad14)
- A1 pad 31: unconnected-(A1-SDA/A4-Pad31) -> /SDA
- A1 pad 32: unconnected-(A1-SCL/A5-Pad32) -> /SCL
Routing:
- net /SDA: track 58.0 -> 83.9 mm
- net /SCL: track 63.9 -> 89.8 mm, vias 0 -> 1
- net /RST2: track 54.2 -> 56.2 mm
- net GND: vias 51 -> 57
Other:
- board text added: "Arduino UNO Click shield v${REVISION} by MPro"
- board text removed: "Arduino UNO Click shield v1.0 by MPro"

Commit message: Arduino UNO Click shield v1.2
Parts:
- added JP3: VCC, footprints:SolderJumper-3_P1.3mm_Bridged12_RoundedPad1.0x1.5mm, F.Cu at (104.1, 83.8)
- added JP4: TX, footprints:SolderJumper-2_P1.3mm_Open_RoundedPad1.0x1.5mm, B.Cu at (133.6, 43.7)
- added JP5: RX, footprints:SolderJumper-2_P1.3mm_Open_RoundedPad1.0x1.5mm, B.Cu at (131.1, 43.7)
- added R2: 10k, footprints:R_0805_2012Metric, F.Cu at (119.9, 51.9)
- added TP2: ~, footprints:TestPoint_Pad_D1.0mm, F.Cu at (111.1, 59.6)
- added TP3: TX, footprints:TestPoint_Pad_D1.0mm, F.Cu at (110.9, 54.6)
- added TP4: RX, footprints:TestPoint_Pad_D1.0mm, F.Cu at (111.1, 57.5)
- added TP5: ~, footprints:TestPoint_Pad_D1.0mm, F.Cu at (121.9, 49.9)
- J4: value UPDI -> SWD; footprint footprints:PinHeader_1x03_P1.27mm_Vertical -> footprints:PinHeader_1x04_P2.54mm_Horizontal
- R1: value 470 -> 10k
- U1: value ATtiny1616-M -> PY32F030F18P6TU; footprint footprints:VQFN-20-1EP_3x3mm_P0.4mm_EP1.7x1.7mm -> Package_SO:TSSOP-20_4.4x6.5mm_P0.65mm
- moved J4 56.0 mm to (126.8, 42.5), turned to 0 degrees
- moved LOGO3 18.4 mm to (80.6, 82.9)
- moved LOGO2 14.6 mm to (89.5, 82.9)
- moved C1 2.29 mm to (116.3, 64.6), turned to 0 degrees
- moved C2 1.78 mm to (116.3, 62.6), turned to 0 degrees
- moved R1 1.51 mm to (114.4, 66.6), turned to 180 degrees
- moved U1 0.55 mm to (116.2, 57.7), turned to 0 degrees
- renumbered R2 to R3, R3 to R4
Connections:
- A1 pad 2: VCC -> Net-(A1-IOREF)
- A1 pad 3: unconnected-(A1-~{RESET}-Pad3) -> /~{RST}
- J4 pad 1: Net-(J4-Pin_1) -> GND
- J4 pad 2: GND -> SWD
- J4 pad 3: VCC -> SWCLK
- R1 pad 1: Net-(J4-Pin_1) -> VCC
- R1 pad 2: UPDI -> /~{RST}
- U1 pad 1: /MISO -> /TxD_pass2
- U1 pad 10: unconnected-(U1-PB4-Pad10) -> /MOSI
- U1 pad 11: /RxD2 -> /SCK
- U1 pad 12: /TxD2 -> /~{SS1}
- U1 pad 13: unconnected-(U1-PB1-Pad13) -> /MISO
- U1 pad 14: unconnected-(U1-PB0-Pad14) -> SWD
- U1 pad 15: unconnected-(U1-PC0-Pad15) -> SWCLK
- U1 pad 16: /RxD_pass2 -> unconnected-(U1-PB4-Pad16)
- U1 pad 17: /TxD_pass2 -> unconnected-(U1-PB5-Pad17)
- U1 pad 18: unconnected-(U1-PC3-Pad18) -> /TxD2
- U1 pad 19: UPDI -> /RxD2
- U1 pad 2: /SCK -> /RxD_pass2
- U1 pad 20: /MOSI -> Net-(U1-PF4/BOOT0)
- U1 pad 3: GND -> /~{RST}
- U1 pad 4: VCC -> unconnected-(U1-PF3-Pad4)
- U1 pad 5: /~{SS1} -> Net-(U1-PA2)
- U1 pad 6: unconnected-(U1-PA5-Pad6) -> Net-(U1-PA3)
- U1 pad 7: unconnected-(U1-PA6-Pad7) -> GND
- U1 pad 8: unconnected-(U1-PA7-Pad8) -> Net-(U1-PB2)
- U1 pad 9: unconnected-(U1-PB5-Pad9) -> VCC
Routing:
- net /~{RST}: track 0.00 -> 48.1 mm, vias 0 -> 2
- net Net-(J4-Pin_1): track 34.3 -> 0.00 mm
- net SWD: track 0.00 -> 21.4 mm
- net SWCLK: track 0.00 -> 18.5 mm
- net /RxD_pass2: track 29.7 -> 43.3 mm
- net /RxD2: track 11.7 -> 25.2 mm
- net /TxD2: track 17.2 -> 30.6 mm
- net GND: track 13.3 -> 4.17 mm, vias 57 -> 72
- net UPDI: track 7.38 -> 0.00 mm, vias 2 -> 0
- net /TxD_pass2: track 28.4 -> 35.4 mm
- net +3.3V: track 51.1 -> 58.1 mm, vias 1 -> 4
- net Net-(U1-PF4/BOOT0): track 0.00 -> 6.75 mm
- net VCC: track 66.2 -> 71.8 mm
- net /MISO: track 89.6 -> 94.9 mm, vias 1 -> 2
- net Net-(U1-PA2): track 0.00 -> 4.34 mm
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Other:
- board text removed: "JLCJLCJLCJLC"
