File: CAN_Click/CAN_Click.kicad_pcb (KiCad board)
At the start: 2 copper layers, 25.4 x 42.9 mm, 25 parts, among them J1 CAN, J2 CAN Click v1.0 by MPro, U1 MCP2515-xST, U2 COS1042T/3, Y1 16MHz

Commit message: quartz changed to 12MHz
Parts:
- C1, C2: value 22pF -> 20pF
- Y1: value 16MHz -> 12MHz
Changed lines of the file:
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@@
 			)
 		)
-		(property "LCSC" "-----"
+		(property "LCSC" "C5383111"
 			(at 0 0 90)
 			(unlocked yes)
@@
 			)
 		)
-		(property "LCSC" "-----"
+		(property "LCSC" "C5383112"
 			(at 0 0 90)
 			(unlocked yes)
@@
 			)
 		)
-		(property "Value" "16MHz"
+		(property "Value" "12MHz"
 			(at 0 2.450001 90)
 			(layer "F.Fab")
@@
 			)
 		)
-		(property "LCSC" "C5380579"
+		(property "LCSC" "C9002"
 			(at 0 0 270)
 			(unlocked yes)
@@
 			)
 		)
-		(property "Value" "22pF"
+		(property "Value" "20pF"
 			(at 0 1.679999 0)
 			(layer "F.Fab")
@@
 			)
 		)
-		(property "LCSC" "C1804"
+		(property "LCSC" "C1798"
 			(at 0 0 0)
 			(unlocked yes)
@@
 			)
 		)
-		(property "Value" "22pF"
+		(property "Value" "20pF"
 			(at 0 1.679999 0)
 			(layer "F.Fab")
@@
 			)
 		)
-		(property "LCSC" "C1804"
+		(property "LCSC" "C1798"
 			(at 0 0 180)
 			(unlocked yes)
@@
 			(keep_text_aligned yes)
 		)
-		(gr_text "42,93 mm"
+		(gr_text "42.93 mm"
 			(at 88.258 67.118 90)
 			(layer "Dwgs.User")
@@
 			(keep_text_aligned yes)
 		)
-		(gr_text "25,4 mm"
+		(gr_text "25.4 mm"
 			(at 103.4385 43.173 0)
 			(layer "Dwgs.User")
@@
 			(keep_text_aligned yes)
 		)
-		(gr_text "22,86 mm"
+		(gr_text "22.86 mm"
 			(at 102.1685 89.401 0)
 			(layer "Dwgs.User")
