File: I2C_1-Wire_Click/I2C_1-Wire_Click.kicad_pcb (KiCad board)
At the start: 2 copper layers, 25.4 x 42.9 mm, 19 parts, among them J1 I^{2}C to 1-Wire Click v1.0 b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, J2 1-Wire, Q1 BSS84, U1 DS2482-100

Commit message: project files updated to Kicad version 9.0.1
Parts:
- J1: value I^{2}C to 1-Wire Click v1.0 by MPro -> I^{2}C to 1-Wire Click v${REVISION} by MPro

Commit message: updated 3D models and project files
Other:
- board text removed: "JLCJLCJLCJLC"
Changed lines of the file:
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@@
 			)
 		)
-		(model "${KIPRJMOD}/shapes3D/Jumper-blue.step"
+		(model "${KIPRJMOD}/shapes3D/Jumper-blue.stpZ"
 			(offset
 				(xyz 0 -3.81 0)
@@
 			)
 		)
-		(model "${KIPRJMOD}/shapes3D/Jumper-red.step"
+		(model "${KIPRJMOD}/shapes3D/Jumper-red.stpZ"
 			(offset
 				(xyz 0 -1.27 0)
@@
 			)
 		)
-		(model "${KIPRJMOD}/shapes3D/Jumper-blue.step"
+		(model "${KIPRJMOD}/shapes3D/Jumper-blue.stpZ"
 			(offset
 				(xyz 0 -3.81 0)
@@
 		(embedded_fonts no)
 	)
-	(gr_text "JLCJLCJLCJLC"
-		(at 113.03 86.36 0)
-		(layer "B.SilkS")
-		(effects
-			(font
-				(size 0.81 0.81)
-				(thickness 0.15)
-				(bold yes)
-			)
-			(justify left bottom mirror)
-		)
-	)
 	(dimension
 		(type aligned)
@@
 			(prefix "")
 			(suffix "")
-			(units 3)
+			(units 2)
 			(units_format 1)
-			(precision 4)
+			(precision 2)
 		)
 		(style
@@
 			(keep_text_aligned yes)
 		)
-		(gr_text "22,8600 mm"
+		(gr_text "22,86 mm"
 			(at 101.551 88.171 0)
 			(layer "Dwgs.User")
@@
 			(prefix "")
 			(suffix "")
-			(units 3)
+			(units 2)
 			(units_format 1)
-			(precision 4)
+			(precision 2)
 		)
 		(style
@@
 			(keep_text_aligned yes)
 		)
-		(gr_text "42,9260 mm"
+		(gr_text "42,93 mm"
 			(at 86.431 65.318 90)
 			(layer "Dwgs.User")
@@
 			(prefix "")
 			(suffix "")
-			(units 3)
+			(units 2)
 			(units_format 1)
-			(precision 4)
+			(precision 2)
 		)
 		(style
@@
 			(keep_text_aligned yes)
 		)
-		(gr_text "25,4000 mm"
+		(gr_text "25,40 mm"
 			(at 102.821 40.546 0)
 			(layer "Dwgs.User")

Commit message: HW rev 1.1 [corrected error in transistor Q1 connections]
Parts:
- moved R4 12.4 mm to (109.9, 57.6), turned to 0 degrees
- moved Q1 12.3 mm to (109.9, 60.8)
- moved C1 2.21 mm to (98.6, 60.0)
- moved U1 2.21 mm to (103.8, 60.9)
Connections:
- Q1 pad 2: Net-(J2-Pin_1) -> Net-(Q1-S)
- Q1 pad 3: Net-(Q1-D) -> Net-(J2-Pin_1)
- R4 pad 2: Net-(Q1-D) -> Net-(Q1-S)
Routing:
- net Net-(Q1-G): track 31.8 -> 2.59 mm
- net Net-(J2-Pin_1): track 26.4 -> 21.3 mm
- net Net-(Q1-S): track 0.00 -> 4.09 mm
- net Net-(Q1-D): track 2.66 -> 0.00 mm
- net VCC: track 46.5 -> 48.7 mm
- net Net-(JP5-C): track 10.1 -> 8.70 mm
- net Net-(J1-SCL): track 24.4 -> 23.3 mm
- net Net-(J1-SDA): track 26.7 -> 27.6 mm
- net GND: track 4.13 -> 4.30 mm, vias 17 -> 19
