File: OpenTherm_Click/OpenTherm_Click.kicad_pcb (KiCad board)
At the start: 2 copper layers, 25.4 x 57.2 mm, 58 parts, among them J1 BOILER, J2 THERM, J3 OpenTherm Click v1.0 by MPro, Q1 MMBT2907A, Q2 MMBT2907A, Q3 MMBT2907A, Q4 MMBT2907A, Q5 MMBT2222A, Q6 MMBT2222A, U1 MT3540-F23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

Commit message: RxB LED brightness adjusted
Parts:
- R17: value 1k8 -> 5k1
Changed lines of the file:
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@@
 			)
 		)
-		(property "Value" "1k8"
+		(property "Value" "5k1"
 			(at 0 1.43 0)
 			(layer "F.Fab")
@@
 			)
 		)
-		(property "LCSC" "C4177"
+		(property "LCSC" "C23186"
 			(at 0 0 180)
 			(unlocked yes)
