File: OpenTherm_Click/OpenTherm_Click.kicad_sch (KiCad schematic)
At the start: 55 parts, among them J1 BOILER, J2 THERM, J3 OpenTherm Click v${REVISION} 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, Q1 MMBT2907A, Q2 MMBT2907A, Q3 MMBT2907A, Q4 MMBT2907A, Q5 MMBT2222A, Q6 MMBT2222A, U1 MT3540-F23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

Commit message: RxB LED brightness adjusted
Parts:
- R17: value 1k8 -> 5k1; LCSC C4177 -> C23186
Changed lines of the file:
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@@
 	(title_block
 		(title "OpenTherm Click")
-		(date "2025-07-10")
+		(date "2025-09-14")
 		(rev "1.0")
 		(company "© 2025 MPro")
@@
 			)
 		)
-		(property "Value" "1k8"
+		(property "Value" "5k1"
 			(at 201.93 121.666 90)
 			(effects
@@
 			)
 		)
-		(property "LCSC" "C4177"
+		(property "LCSC" "C23186"
 			(at 201.93 119.38 90)
 			(effects
